File: Reflow-Oven.kicad_sch (KiCad schematic)
At the start: 53 parts, among them J1 Thermocouple 1, J10 Display, J11 GND(A), J12 +12V, J13 Servo 2, J14 Servo 1, J15 Door, J17 Servo 3, J18 Ambient snesor, J19 Controls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

Commit message: Single servo with cutoff
Parts:
- removed C4: 1000uf, Capacitor_SMD:CP_Elec_10x10.5, symbol Device:C_Polarized
- removed J11: GND(A), Connector_Wire:SolderWirePad_1x01_SMD_5x10mm, symbol Connector:Conn_01x01_Pin
- removed J12: +12V, Connector_Wire:SolderWirePad_1x01_SMD_5x10mm, symbol Connector:Conn_01x01_Pin
- removed J13: Servo 2, Connector_PinHeader_2.54mm:PinHeader_1x03_P2.54mm_Vertical_SMD, symbol Connector:Conn_01x03_Pin
- removed J17: Servo 3, Connector_PinHeader_2.54mm:PinHeader_1x03_P2.54mm_Vertical_SMD, symbol Connector:Conn_01x03_Pin
- removed J20: Servo 4, Connector_PinHeader_2.54mm:PinHeader_1x03_P2.54mm_Vertical_SMD, symbol Connector:Conn_01x03_Pin
- removed J5: Fan, Connector_PinHeader_2.54mm:PinHeader_1x04_P2.54mm_Vertical_SMD, symbol Connector:Conn_01x04_Pin
- removed R31: 1K, Resistor_SMD:R_1206_3216Metric_Pad1.30x1.75mm_HandSolder, symbol Device:R
- removed R33, R35, R36: 220R, Resistor_SMD:R_1206_3216Metric_Pad1.30x1.75mm_HandSolder, symbol Device:R
- added C20: 10nf, Capacitor_SMD:C_1206_3216Metric_Pad1.33x1.80mm_HandSolder, symbol Device:C
- added J16: Door, Connector_PinHeader_2.54mm:PinHeader_1x02_P2.54mm_Vertical_SMD, symbol Connector:Conn_01x02_Pin
- added Q4: AO3401A, PMV20XNER:SOT23-TO-236AB_NEX, symbol Transistor_FET:AO3401A
- added R15: 4K7, Resistor_SMD:R_1206_3216Metric_Pad1.30x1.75mm_HandSolder, symbol Device:R
- added R5: 330R, Resistor_SMD:R_1206_3216Metric, symbol Device:R
- added R6: 10K, Resistor_SMD:R_1206_3216Metric, symbol Device:R
Connections:
- net +3.3V: now also R15.2
- net +5V: now also Q4.2 (S), R6.2; no longer C10.1, J14.2 (Pin_2)
- net GND: now also C20.1, J16.2 (Pin_2)
- net Door CL: now reaches U1.32 (GPIO27_ADC1)
- net Door CL: now also C20.2, J16.1 (Pin_1), R15.1
- net Door renamed Door OP
- net Servo 1 renamed Servo EN
- net Servo EN: now also R5.1; no longer R32.1
- net Servo 2 renamed Servo SIG
- net Servo SIG: now also R32.1
- net Servo 3: no longer names the net of U1.6 (GPIO4)
- net Servo 4: no longer names the net of U1.7 (GPIO5)
- new net: C10.1, J14.2 (Pin_2), Q4.3 (D)
- new net: Q4.1 (G), R5.2, R6.1
Other:
- moved on the sheet: C10, C3, J14, R32

Commit message: Updated
Parts:
- added C18, C21: 100nf, Capacitor_SMD:C_1210_3225Metric_Pad1.33x2.70mm_HandSolder, symbol Device:C
- added C2: 220uf, Capacitor_SMD:CP_Elec_8x10.5, symbol Device:C_Polarized
- added C4: 1000uf, Capacitor_SMD:CP_Elec_10x10.5, symbol Device:C_Polarized
- added D1: 1N5819WS, Diode_SMD:D_SOD-323_HandSoldering, symbol Diode:1N5819WS
- added J11: GND(A), Connector_Wire:SolderWirePad_1x01_SMD_5x10mm, symbol Connector:Conn_01x01_Pin
- added J12: +12V, Connector_Wire:SolderWirePad_1x01_SMD_5x10mm, symbol Connector:Conn_01x01_Pin
- added J17: SSR Temp, Connector_PinHeader_2.54mm:PinHeader_1x03_P2.54mm_Vertical_SMD, symbol Connector:Conn_01x03_Pin
- added J20: Fan, Connector_PinHeader_2.54mm:PinHeader_1x04_P2.54mm_Vertical_SMD, symbol Connector:Conn_01x04_Pin
- added R16, R17: 4K7, Resistor_SMD:R_1206_3216Metric, symbol Device:R
- J15: value Door -> Door OP
- J16: value Door -> Door CL
- J8: value Conn_01x02_Pin -> SSR1
- J9: value Conn_01x02_Pin -> SSR2
- R14, R15, R21, R24, R29, R32, R34: footprint Resistor_SMD:R_1206_3216Metric_Pad1.30x1.75mm_HandSolder -> Resistor_SMD:R_1206_3216Metric
Connections:
- net +3.3V: now also C18.1, C2.1, C21.1, J17.1 (Pin_1), R16.2, R17.2
- net Door CL: now also U1.7 (GPIO5); no longer U1.32 (GPIO27_ADC1)
- net Door OP: now also U1.6 (GPIO4); no longer U1.31 (GPIO26_ADC0)
- net GND: now also C18.2, C2.2, C21.2, C4.2, D1.2 (A), J11.1 (Pin_1), J17.3 (Pin_3), J20.3 (Pin_3)
- net at U1.34 (GPIO28_ADC2): now also J20.2 (Pin_2), R16.1
- new net: J20.1 (Pin_1), U1.32 (GPIO27_ADC1)
- new net: J17.2 (Pin_2), R17.1, U1.31 (GPIO26_ADC0)
- new net +12V: C4.1, D1.1 (K), J12.1 (Pin_1), J20.4 (Pin_4)
